File: pcb/rollscanner.kicad_sch (KiCad schematic)
At the start: 21 parts, among them J1 DIN-5, Q0 Q_NPN, Q1 Q_Photo_NPN, Q2 Q_Photo_NPN, Q3 Q_Photo_NPN, Q4 Q_Photo_NPN, U1 STM32G431C8Tx, U2 ADG706BRUZ, U3 ADG706BRUZ, U4 ADG706BRUZ, U5 ADG706BRUZ, U6 ADG706BRUZ, U7 ADG706BRUZ, U8 ADG706BRUZ

Commit message: a
Parts:
- added A1: Pololu_Breakout_A4988, Module:Pololu_Breakout-16_15.2x20.3mm, symbol Driver_Motor:Pololu_Breakout_A4988
- added J2: Conn_01x04, symbol Connector_Generic:Conn_01x04
Connections:
- net +3.3V: now also A1.2 (VDD)
- net GND: now also A1.1 (GND), A1.7 (GND)
- new net: A1.3 (1B), J2.1 (Pin_1)
- new net: A1.4 (1A), J2.2 (Pin_2)
- new net: A1.5 (2A), J2.3 (Pin_3)
- new net: A1.6 (2B), J2.4 (Pin_4)
- new net +12V: A1.8 (VMOT)
- new net ~{MOTOR_ENABLE}: A1.9 (~{ENABLE})
- new net ~{MOTOR_RESET}: A1.13 (~{RESET})
- new net ~{MOTOR_SLEEP}: A1.14 (~{SLEEP})

Commit message: Update rollscanner.kicad_sch
Parts:
- removed J1: DIN-5, symbol Connector:DIN-5
- removed J2: Conn_01x04, symbol Connector_Generic:Conn_01x04
- removed U2, U3, U4, U5, U6, U7, U8: ADG706BRUZ, ADG706BRUZ:SOP65P640X120-28N, symbol symbols:ADG706BRUZ
- added A2: Pololu_Breakout_A4988, Module:Pololu_Breakout-16_15.2x20.3mm, symbol Driver_Motor:Pololu_Breakout_A4988
- added C1, C2: 10pF, symbol Device:C
- added J2: DIN-5_180degree, symbol Connector:DIN-5_180degree
- added M1, M2: Stepper_Motor_bipolar, symbol Motor:Stepper_Motor_bipolar
- added U10, U11, U12, U2, U3, U4, U5, U6, U7, U8, U9: 74HC165, symbol 74xx:74HC165
- added Y1: 25 MHz, symbol Device:Crystal
Connections:
- net +12V: now also A2.8 (VMOT)
- net +3.3V: now also A2.2 (VDD), U10.16 (VCC), U11.16 (VCC), U12.16 (VCC), U2.16 (VCC), U3.16 (VCC), U4.16 (VCC), U5.16 (VCC), U6.16 (VCC), U7.16 (VCC), U8.16 (VCC), U9.16 (VCC)
- net GND: now also A2.1 (GND), A2.7 (GND), C1.2, C2.2, J2.2, U10.8 (GND), U11.8 (GND), U12.8 (GND), U2.8 (GND), U3.8 (GND), U4.8 (GND), U5.8 (GND), U6.8 (GND), U7.8 (GND), U8.8 (GND), U9.8 (GND)
- net N1: now also U10.11 (D0), U11.11 (D0), U12.11 (D0), U2.11 (D0), U3.11 (D0), U4.11 (D0), U5.11 (D0), U6.11 (D0), U7.11 (D0), U8.11 (D0), U9.11 (D0)
- net N2: now also U10.12 (D1), U11.12 (D1), U12.12 (D1), U2.12 (D1), U3.12 (D1), U4.12 (D1), U5.12 (D1), U6.12 (D1), U7.12 (D1), U8.12 (D1), U9.12 (D1)
- net N3: now also U10.13 (D2), U11.13 (D2), U12.13 (D2), U2.13 (D2), U3.13 (D2), U4.13 (D2), U5.13 (D2), U6.13 (D2), U7.13 (D2), U8.13 (D2), U9.13 (D2)
- net N4: now also U10.14 (D3), U11.14 (D3), U12.14 (D3), U2.14 (D3), U3.14 (D3), U4.14 (D3), U5.14 (D3), U6.14 (D3), U7.14 (D3), U8.14 (D3), U9.14 (D3)
- net N5: now also U10.3 (D4), U11.3 (D4), U12.3 (D4), U2.3 (D4), U3.3 (D4), U4.3 (D4), U5.3 (D4), U6.3 (D4), U7.3 (D4), U8.3 (D4), U9.3 (D4)
- net N6: now also U10.4 (D5), U11.4 (D5), U12.4 (D5), U2.4 (D5), U3.4 (D5), U4.4 (D5), U5.4 (D5), U6.4 (D5), U7.4 (D5), U8.4 (D5), U9.4 (D5)
- net N7: now also U10.5 (D6), U11.5 (D6), U12.5 (D6), U2.5 (D6), U3.5 (D6), U4.5 (D6), U5.5 (D6), U6.5 (D6), U7.5 (D6), U8.5 (D6), U9.5 (D6)
- net N8: now also U10.6 (D7), U11.6 (D7), U12.6 (D7), U2.6 (D7), U3.6 (D7), U4.6 (D7), U5.6 (D7), U6.6 (D7), U7.6 (D7), U8.6 (D7), U9.6 (D7)
- net ~{MOTOR_ENABLE}: now also A2.9 (~{ENABLE}); no longer A1.9 (~{ENABLE})
- net ~{MOTOR_RESET}: now also A2.13 (~{RESET}); no longer A1.13 (~{RESET})
- net ~{MOTOR_SLEEP}: now also A2.14 (~{SLEEP}); no longer A1.14 (~{SLEEP})
- net at A1.3 (1B): now also M1.2 (-)
- net at A1.4 (1A): now also M1.1
- net at A1.5 (2A): now also M1.3
- net at A1.6 (2B): now also M1.4
- net at R6.1: now also J2.5
- net MOTOR1_STEP: now reaches A1.15 (STEP)
- net MOTOR1_DIR: now reaches A1.16 (DIR)
- net at R5.2: now also J2.4
- new net: U6.9 (Q7), U7.10 (DS)
- new net: U7.9 (Q7), U8.10 (DS)
- new net: U2.9 (Q7), U3.10 (DS)
- new net: U3.9 (Q7), U4.10 (DS)
- new net: U4.9 (Q7), U5.10 (DS)
- new net: C1.1, Y1.1
- new net: C2.1, Y1.2
- new net: U8.9 (Q7), U9.10 (DS)
- new net: U10.10 (DS), U9.9 (Q7)
- new net: U5.9 (Q7), U6.10 (DS)
- new net: A2.3 (1B), M2.2 (-)
- new net: A2.4 (1A), M2.1
- new net: A2.5 (2A), M2.3
- new net: A2.6 (2B), M2.4
- new net: U11.9 (Q7), U12.10 (DS)
- new net: U10.9 (Q7), U11.10 (DS)
- new net LOAD_NOTES: U10.1 (~{PL}), U11.1 (~{PL}), U12.1 (~{PL}), U2.1 (~{PL}), U3.1 (~{PL}), U4.1 (~{PL}), U5.1 (~{PL}), U6.1 (~{PL}), U7.1 (~{PL}), U8.1 (~{PL}), U9.1 (~{PL})
- new net NOTE_CLOCK: U10.2 (CP), U11.2 (CP), U12.2 (CP), U2.2 (CP), U3.2 (CP), U4.2 (CP), U5.2 (CP), U6.2 (CP), U7.2 (CP), U8.2 (CP), U9.2 (CP)
- new net NOTE_CLOCK_ENABLE: U10.15 (~{CE}), U11.15 (~{CE}), U12.15 (~{CE}), U2.15 (~{CE}), U3.15 (~{CE}), U4.15 (~{CE}), U5.15 (~{CE}), U6.15 (~{CE}), U7.15 (~{CE}), U8.15 (~{CE}), U9.15 (~{CE})
- new net NOTE_DATA_IN: U12.9 (Q7)
- new net ~{MOTOR1_ENABLE}: A1.9 (~{ENABLE})
- new net ~{MOTOR1_RESET}: A1.13 (~{RESET})
- new net ~{MOTOR1_SLEEP}: A1.14 (~{SLEEP})
- no-connect marks 2 -> 14
Other:
- moved on the sheet: Q0, Q1, Q2, Q3, Q4, R1, R2, R3, R4, R5, R6, R7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

Commit message: y
Parts:
- added C3, C4, C5: 100nF, symbol Device:C
- added C6: 1μF, symbol Device:C
- Y1: footprint (none) -> Crystal:Crystal_SMD_HC49-SD
Connections:
- net +3.3V: now also C3.1, C4.1, C5.1, C6.1
- net GND: now also C3.2, C4.2, C5.2, C6.2
- net at C1.1, Y1.1: now also U1.5 (PF0)
- net at C2.1, Y1.2: now also U1.6 (PF1)
Other:
- moved on the sheet: J2, Q0, Q1, Q2, Q3, Q4, R1, R2, R3, R4, R5, R6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

Commit message: w
Parts:
- removed Q0: Q_NPN, symbol Device:Q_NPN
- removed Q1, Q2, Q3, Q4: Q_Photo_NPN, symbol Device:Q_Photo_NPN
- removed R1, R2, R3, R4: R_US, symbol Device:R_US
- removed U10, U11, U12, U2, U3, U4, U5, U6, U7, U8, U9: 74HC165, symbol 74xx:74HC165
- added C7: 100nF, symbol Device:C
- added D3: CMS06, Diode_SMD:D_SOD-128, symbol Device:D_Schottky
- added J1: USB_C_Receptacle, symbol Connector:USB_C_Receptacle
- added J3: Actuator Solenoid, Connector_PinHeader_2.54mm:PinHeader_1x02_P2.54mm_Vertical, symbol Connector_Generic:Conn_01x02
- added J4: Conn_ST_STDC14, symbol Connector:Conn_ST_STDC14
- added Q5: IRF530NPBF, symbol Transistor_FET:Q_NMOS_GDS
- added R10, R11: 10kΩ, symbol Device:R_US
- added R18: 220Ω, Resistor_SMD:R_0603_1608Metric_Pad0.98x0.95mm_HandSolder, symbol Device:R_US
- added R8, R9: 5.1kΩ, symbol Device:R_US
- added U14: SN74LV1T34DBV, Package_TO_SOT_SMD:SOT-23-5, symbol Logic_LevelTranslator:SN74LV1T34DBV
- R7: value 10kΩ -> 220Ω
Connections:
- net ~{MOTOR_ENABLE} is gone; now on net ~{MOTOR2_ENABLE}: A2.9 (~{ENABLE})
- net ~{MOTOR_RESET} is gone; now on net ~{MOTOR2_RESET}: A2.13 (~{RESET})
- net ~{MOTOR_SLEEP} is gone; now on net ~{MOTOR2_SLEEP}: A2.14 (~{SLEEP})
- net +12V: now also D3.1 (K), J3.1 (Pin_1)
- net +3.3V: now also U1.20 (VREF+), J4.3 (VCC), R10.2
- net +5V: now also U14.5 (VCC)
- net GND: now also C7.2, J1.A1 (GND), J1.A12 (GND), J1.B1 (GND), J1.B12 (GND), J1.S1 (SHIELD), J4.11 (GNDDetect), J4.5 (GND), J4.7 (GND), Q5.3 (S), R11.1, R8.1, R9.2, U14.3 (GND)
- net MOTOR1_DIR: now also U1.45 (PB8), R11.2
- net MOTOR1_STEP: now also U1.30 (PA8)
- net ~{MOTOR1_ENABLE}: now also U1.44 (PB7)
- net ~{MOTOR1_RESET}: now also U1.42 (PB5)
- net ~{MOTOR1_SLEEP}: now also U1.43 (PB6)
- net V_COM_TX: now reaches U1.10 (PA2)
- net V_COM_TX: now also J4.13 (VCP_RX)
- net V_COM_RX: now reaches U1.11 (PA3)
- net V_COM_RX: now also J4.14 (VCP_TX)
- net at U1.14 (PA6): now also R18.2
- net MOTOR2_MS1: now reaches U1.16 (PB0)
- net MOTOR2_MS1: now also A2.10 (MS1)
- net MOTOR2_MS2: now reaches U1.17 (PB1)
- net MOTOR2_MS2: now also A2.11 (MS2)
- net MOTOR2_MS3: now reaches U1.18 (PB2)
- net MOTOR2_MS3: now also A2.12 (MS3)
- net MOTOR1_MS2: now reaches U1.22 (PB10)
- net MOTOR1_MS2: now also A1.11 (MS2)
- net MOTOR1_MS3: now reaches U1.25 (PB11)
- net MOTOR1_MS3: now also A1.12 (MS3)
- net ~{MOTOR2_RESET}: now reaches U1.26 (PB12)
- net ~{MOTOR2_SLEEP}: now reaches U1.27 (PB13)
- net ~{MOTOR2_ENABLE}: now reaches U1.28 (PB14)
- net MOTOR2_DIR: now reaches U1.29 (PB15)
- net MOTOR2_DIR: now also A2.16 (DIR)
- net at U1.31 (PA9): now also R7.2
- net at U1.33 (PA11): now also J1.A7 (D-), J1.B7 (D-)
- net at U1.34 (PA12): now also J1.A6 (D+), J1.B6 (D+)
- net JTMS/SWDIO: now reaches U1.37 (PA13)
- net JTMS/SWDIO: now also J4.4 (JTMS/SWDIO)
- net JTCK/SWCLK: now reaches U1.38 (PA14)
- net JTCK/SWCLK: now also J4.6 (JCLK/SWCLK)
- net JTDI: now reaches U1.39 (PA15)
- net JTDI: now also J4.10 (JTDI/NC)
- net JTDO/SWO: now reaches U1.40 (PB3)
- net JTDO/SWO: now also J4.8 (JTDO/SWO)
- net MOTOR1_MS1: now reaches U1.46 (PB9)
- net MOTOR1_MS1: now also A1.10 (MS1)
- net ~{RST}: now reaches U1.7 (PG10)
- net ~{RST}: now also J4.12 (~{RST}), R10.1
- net MOTOR2_STEP: now reaches U1.8 (PA0)
- net MOTOR2_STEP: now also A2.15 (STEP)
- net at R7.1: now also U14.2 (A)
- net at R6.2: now also U14.4 (Y)
- new net: Q5.1 (G), R18.1
- new net: D3.2 (A), J3.2 (Pin_2), Q5.2 (D)
- new net: C7.1, J1.A4 (VBUS), J1.A9 (VBUS), J1.B4 (VBUS), J1.B9 (VBUS)
- new net: J1.A5 (CC1), R8.2
- new net: J1.B5 (CC2), R9.1
Other:
- added sheet Light Sensors (phototransistors.kicad_sch)
- added sheet Regulators (voltage_regulators.kicad_sch)
- added sheet Shift Registers (shift_registers.kicad_sch)
- note added: "Tx and Rx Swapped!"
- moved on the sheet: A1, A2, C1, C2, C3, C4, C5, C6, J2, M1, M2, R5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
